File: s2/kicad/knobs_2x5/knobs_2x5/knobs_2x5.kicad_pcb (KiCad board)
At the start: 2 copper layers, 95 x 46 mm, 11 parts, among them J1 Conn_02x08_Odd_Even

Commit message: added kicad projects
Connections:
- net +5V renamed +3.3V
Other:
- board text added: "3.3 V"
- board text removed: "5v"
